Commit message: minor changes to solve launch files

File: daVinciCore/urdf/daVinci_exp.urdf.xacro (robot description, xacro)
@@ -18,5 +18,5 @@
       <origin rpy="0 0 0" xyz="0 0 0"/>
       <geometry>
-	<mesh filename="package://daVinci/meshes/slave_frame.stl"/>
+	<mesh filename="package://daVinciCore/meshes/slave_frame.stl"/>
       </geometry>
     </visual>
@@ -24,5 +24,5 @@
       <origin rpy="0 0 0" xyz="0 0 1.0"/>
       <geometry>
-	<mesh filename="package://daVinci/meshes/slave_frame.stl"/>
+	<mesh filename="package://daVinciCore/meshes/slave_frame.stl"/>
       </geometry>
     </collision>
@@ -52,5 +52,5 @@
 	      <origin rpy="0 0 0" xyz="0 0 0"/>
 	      <geometry>
-		<mesh filename="package://daVinci/meshes/mounting_base.stl"/>
+		<mesh filename="package://daVinciCore/meshes/mounting_base.stl"/>
 	      </geometry>
 	      <material name="green">
@@ -61,5 +61,5 @@
 	      <origin rpy="0 0 0" xyz="0 0 0"/>
 	      <geometry>
-		<mesh filename="package://daVinci/meshes/mounting_base.stl"/>
+		<mesh filename="package://daVinciCore/meshes/mounting_base.stl"/>
 	      </geometry>
 	    </collision>
@@ -81,5 +81,5 @@
 	      <origin rpy="0 0 0" xyz="0.001 -0.1 -0.1375"/>
 	      <geometry>
-		<mesh filename="package://daVinci/meshes/outer_yaw.stl"/>
+		<mesh filename="package://daVinciCore/meshes/outer_yaw.stl"/>
 	      </geometry>
 	      <material name="red">
@@ -90,5 +90,5 @@
 	      <origin rpy="0 0 0" xyz="0.001 -0.1 -0.1375"/>
 	      <geometry>
-		<mesh filename="package://daVinci/meshes/outer_yaw.stl"/>
+		<mesh filename="package://daVinciCore/meshes/outer_yaw.stl"/>
 	      </geometry>
 	    </collision>
@@ -110,5 +110,5 @@
 	      <origin rpy="0 0 0" xyz="-0.040 -0.130 -0.0901"/>
 	      <geometry>
-		<mesh filename="package://daVinci/meshes/outer_pitch_base.stl"/>
+		<mesh filename="package://daVinciCore/meshes/outer_pitch_base.stl"/>
 	      </geometry>
 	      <material name="blue">
@@ -119,5 +119,5 @@
 	      <origin rpy="0 0 0" xyz="-0.040 -0.130 -0.0901"/>
 	      <geometry>
-		<mesh filename="package://daVinci/meshes/outer_pitch_base.stl"/>
+		<mesh filename="package://daVinciCore/meshes/outer_pitch_base.stl"/>
 	      </geometry>
 	    </collision>
@@ -139,5 +139,5 @@
 	      <origin rpy="0 0 0" xyz="0 -0.066 -0.010"/>
 	      <geometry>
-		<mesh filename="package://daVinci/meshes/outer_pitch_front.stl"/>
+		<mesh filename="package://daVinciCore/meshes/outer_pitch_front.stl"/>
 	      </geometry>
 	      <material name="red"/>
@@ -146,5 +146,5 @@
 	      <origin rpy="0 0 0" xyz="0 -0.066 -0.010"/>
 	      <geometry>
-		<mesh filename="package://daVinci/meshes/outer_pitch_front.stl"/>
+		<mesh filename="package://daVinciCore/meshes/outer_pitch_front.stl"/>
 	      </geometry>
 	    </collision>
@@ -166,5 +166,5 @@
 	      <origin rpy="0 0 0" xyz="0 -0.093 -0.010"/>
 	      <geometry>
-		<mesh filename="package://daVinci/meshes/outer_pitch_bottom.stl"/>
+		<mesh filename="package://daVinciCore/meshes/outer_pitch_bottom.stl"/>
 	      </geometry>
 	      <material name="green"/>
@@ -173,5 +173,5 @@
 	      <origin rpy="0 0 0" xyz="0 -0.093 -0.010"/>
 	      <geometry>
-		<mesh filename="package://daVinci/meshes/outer_pitch_bottom.stl"/>
+		<mesh filename="package://daVinciCore/meshes/outer_pitch_bottom.stl"/>
 	      </geometry>
 	    </collision>
@@ -193,5 +193,5 @@
 	      <origin rpy="0 0 0" xyz="0 -0.093 -0.010"/>
 	      <geometry>
-		<mesh filename="package://daVinci/meshes/outer_pitch_top.stl"/>
+		<mesh filename="package://daVinciCore/meshes/outer_pitch_top.stl"/>
 	      </geometry>
 	      <material name="green"/>
@@ -200,5 +200,5 @@
 	      <origin rpy="0 0 0" xyz="0 -0.093 -0.010"/>
 	      <geometry>
-		<mesh filename="package://daVinci/meshes/outer_pitch_top.stl"/>
+		<mesh filename="package://daVinciCore/meshes/outer_pitch_top.stl"/>
 	      </geometry>
 	    </collision>
@@ -220,5 +220,5 @@
 	      <origin rpy="0 0 0" xyz="-0.031 -0.086 -0.070"/>
 	      <geometry>
-		<mesh filename="package://daVinci/meshes/outer_insertion.stl"/>
+		<mesh filename="package://daVinciCore/meshes/outer_insertion.stl"/>
 	      </geometry>
 	      <material name="blue"/>
@@ -227,5 +227,5 @@
 	      <origin rpy="0 0 0" xyz="-0.031 -0.086 -0.070"/>
 	      <geometry>
-		<mesh filename="package://daVinci/meshes/outer_insertion.stl"/>
+		<mesh filename="package://daVinciCore/meshes/outer_insertion.stl"/>
 	      </geometry>
 	    </collision>
@@ -248,5 +248,5 @@
 	      <origin rpy="0 0 0" xyz="0 -0.041 0"/>
 	      <geometry>
-		<mesh filename="package://daVinci/meshes/tool_adaptor.stl"/>
+		<mesh filename="package://daVinciCore/meshes/tool_adaptor.stl"/>
 	      </geometry>
 	      <material name="green"/>
@@ -255,5 +255,5 @@
 	      <origin rpy="0 0 0" xyz="0 -0.041 0"/>
 	      <geometry>
-		<mesh filename="package://daVinci/meshes/tool_adaptor.stl"/>
+		<mesh filename="package://daVinciCore/meshes/tool_adaptor.stl"/>
 	      </geometry>
 	    </collision>
@@ -273,5 +273,5 @@
 	      <origin rpy="0 0 0" xyz="0 -0.034 0"/>
 	      <geometry>
-		<mesh filename="package://daVinci/meshes/tool_asm.stl"/>
+		<mesh filename="package://daVinciCore/meshes/tool_asm.stl"/>
 	      </geometry>
 	      <material name="red"/>
@@ -280,5 +280,5 @@
 	      <origin rpy="0 0 0" xyz="0 -0.034 0"/>
 	      <geometry>
-		<mesh filename="package://daVinci/meshes/tool_asm.stl"/>
+		<mesh filename="package://daVinciCore/meshes/tool_asm.stl"/>
 	      </geometry>
 	    </collision>
